Commit message: Added Lidar

File: src/nav_bot/description/nav_bot.urdf.xacro (robot description, xacro)
@@ -2,6 +2,10 @@
 <robot xmlns:xacro="http://www.ros.org/wiki/xacro"  name="nav_bot">
     <!-- <link name="base_link"></link> -->
+    <!-- Robot Structure-->
     <xacro:include filename="structure.xacro"/>
+    <!-- Ros2 Control -->
     <xacro:include filename="ros2_control.xacro"/>
+    <!-- Lidar-->
+    <xacro:include filename="lidar.xacro"/>
 </robot>
 <!--

File: src/nav_bot/description/structure.xacro (robot description, xacro)
@@ -3,15 +3,33 @@
     <xacro:include filename="macro_inertia.xacro"/>
     <!-- Colors -->
-    <material name="white">
-        <color rgba="1 1 1 1" />
+    <material name="black">
+        <color rgba="0.0 0.0 0.0 1.0"/>
+    </material>
+    <material name="dark">
+        <color rgba="0.3 0.3 0.3 1.0"/>
+    </material>
+    <material name="light_black">
+        <color rgba="0.4 0.4 0.4 1.0"/>
+    </material>
+    <material name="blue">
+        <color rgba="0.0 0.0 0.8 1.0"/>
+    </material>
+    <material name="green">
+        <color rgba="0.0 0.8 0.0 1.0"/>
+    </material>
+    <material name="grey">
+        <color rgba="0.5 0.5 0.5 1.0"/>
     </material>
     <material name="orange">
-        <color rgba="1 0.3 0.1 1"/>
+        <color rgba="${255/255} ${108/255} ${10/255} 1.0"/>
     </material>
-    <material name="blue">
-        <color rgba="0.2 0.2 1 1"/>
+    <material name="brown">
+        <color rgba="${222/255} ${207/255} ${195/255} 1.0"/>
     </material>
-    <material name="black">
-        <color rgba="0 0 0 1"/>
+    <material name="red">
+        <color rgba="0.8 0.0 0.0 1.0"/>
+    </material>
+    <material name="white">
+        <color rgba="1.0 1.0 1.0 1.0"/>
     </material>
     <!-- Base Link -->

Commit message: Added Simple Camera and Depth Camera

File: src/nav_bot/description/nav_bot.urdf.xacro (robot description, xacro)
@@ -8,4 +8,8 @@
     <!-- Lidar-->
     <xacro:include filename="lidar.xacro"/>
+    <!-- Camera -->
+    <xacro:include filename="camera.xacro"/>
+    <!-- Depth Camera -->
+    <xacro:include filename="depth_camera.xacro"/>
 </robot>
 <!--

File: src/nav_bot/description/structure.xacro (robot description, xacro)
@@ -50,11 +50,11 @@
         </visual>
         <collision>
-            <origin xyz="0.15 0 0.075"/>
+            <origin xyz="0.225 0 0.025"/>
             <geometry>
-                <box size="0.3 0.3 0.15"/>
+                <box size="0.45 0.3 0.05"/>
             </geometry>
         </collision>
-        <xacro:inertial_box mass="0.5" x="0.3" y="0.3" z="0.15">
-            <origin xyz="0.15 0 0.075" rpy="0 0 0"/>
+        <xacro:inertial_box mass="0.5" x="0.45" y="0.3" z="0.05">
+            <origin xyz="0.225 0 0.025" rpy="0 0 0"/>
         </xacro:inertial_box>
     </link>
