Commit message: Added: * SLAM * Nav2

File: src/nav_bot/description/lidar.xacro (robot description, xacro)
@@ -12,5 +12,5 @@
                 <cylinder radius="0.05" length="0.04"/>
             </geometry>
-            <material name="red"/>
+            <material name="green"/>
         </visual>
         <collision>
@@ -25,5 +25,5 @@
     <!-- Gazebo-->
     <gazebo reference="lidar_body">
-        <material>Gazebo/Red</material>
+        <material>Gazebo/Green</material>
         <sensor name="my_lidar" type="gpu_lidar">
             <pose> 0 0 0 0 0 0 </pose>
@@ -40,5 +40,5 @@
                 <range>
                     <min>0.3</min>
-                    <max>12</max>
+                    <max>10</max>
                 </range>
             </lidar>

File: src/nav_bot/description/structure.xacro (robot description, xacro)
@@ -21,4 +21,7 @@
         <color rgba="0.5 0.5 0.5 1.0"/>
     </material>
+    <material name="yellow">
+        <color rgba="1.0 1.0 0.0 1.0"/>
+    </material>
     <material name="orange">
         <color rgba="${255/255} ${108/255} ${10/255} 1.0"/>
@@ -35,4 +38,11 @@
     <!-- Base Link -->
     <link name="base_link"></link>
+    <!-- Base Footprint -->
+    <joint name="base_footprint_joint" type="fixed">
+        <parent link="base_link"/>
+        <child link="base_footprint"/>
+        <origin xyz="0 0 0" rpy="0 0 0"/>
+    </joint>
+    <link name="base_footprint"></link>
     <!-- CHASSIS LINK-->
     <joint name="chassis_joint" type="fixed">
@@ -47,5 +57,5 @@
                 <box size="0.45 0.3 0.05"/>      <!-- <box size="0.3 0.3 0.15"/> -->
             </geometry>
-            <material name="orange"/>
+            <material name="yellow"/>
         </visual>
         <collision>
@@ -94,5 +104,5 @@
                 <cylinder radius="0.05" length="0.04"/>
             </geometry>
-            <material name="black"/>
+            <material name="blue"/>
         </visual>
         <collision>
@@ -116,5 +126,5 @@
                 <sphere radius="0.05"/>
             </geometry>
-            <material name="blue"/>
+            <material name="red"/>
         </visual>
         <collision>
@@ -151,5 +161,5 @@
                 <sphere radius="0.05"/>
             </geometry>
-            <material name="black"/>
+            <material name="red"/>
         </visual>
         <collision>
