Commit message: Optimized Nav2

File: src/nav_bot/description/camera.xacro (robot description, xacro)
@@ -12,5 +12,5 @@
                 <box size="0.025 0.025 0.025"/>
             </geometry>
-            <material name="brown"/>
+            <material name="red"/>
         </visual>
         <collision>
@@ -31,5 +31,5 @@
     <!-- Gazebo-->
     <gazebo reference="camera_body">
-        <material>Gazebo/Brown</material>
+        <material>Gazebo/Red</material>
         <sensor name="my_camera" type="camera">
             <pose> 0 0 0 0 0 0 </pose>
